File: display_adapter.kicad_pcb (KiCad board)
At the start: 2 copper layers, 36.4 x 68.3 mm, 8 parts, among them J1 Conn_Display, J2 Inky_Left_1_20, J3 Inky_Right_21_40, J4 Ada_SPI_Display

Commit message: Rev 0.90: fix: swap left-right for Inky-Pack
Parts:
- added G***: LOGO, LOGO, B.Cu at (107.5, 106.2)
- moved J3 17.8 mm to (98.6, 148.3)
- moved J2 16.4 mm to (116.4, 100.0)
Routing:
- net /Display_BUSY: track 21.6 -> 34.1 mm
- net /SCLK0: track 26.9 -> 31.6 mm
- net /Display_RST: track 28.1 -> 32.2 mm
- net /Display_DC: track 30.3 -> 28.1 mm
- net GND: track 4.34 -> 6.31 mm
- net +3V3: vias 0 -> 1
Other:
- board text added: "1"
- board text added: "3V3"
- board text added: "40"
- board text added: "Adafruit"
- board text added: "Busy"
- board text added: "CS"
- board text added: "DC"
- board text added: "GND"
- board text added: "MOSI"
- board text added: "Pimoroni Inky-Pack"
- board text added: "RST"
- board text added: "SCLK"
- board text added: "VCC"
- board text added: "https://github.com/bablokb/pcb-pico-datalogger Display Adapter Rev. 0.90"

Commit message: display-adapter: Rev 1.00 ready for production
Other:
- board text added: "https://github.com/bablokb/pcb-pico-datalogger Display Adapter Rev. 1.00"
- board text removed: "https://github.com/bablokb/pcb-pico-datalogger Display Adapter Rev. 0.90"
Changed lines of the file:
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@@
     (property "Sheetname" "")
     (property "exclude_from_bom" "")
-    (attr through_hole exclude_from_bom)
+    (attr through_hole exclude_from_pos_files exclude_from_bom)
     (fp_text reference "J4" (at 0 34) (layer "F.SilkS")
       (effects (font (size 1 1) (thickness 0.15)))
@@
     (property "Sheetname" "")
     (property "exclude_from_bom" "")
-    (attr through_hole exclude_from_bom)
+    (attr through_hole exclude_from_pos_files exclude_from_bom)
     (fp_text reference "J3" (at 0.4 51.55) (layer "F.SilkS")
       (effects (font (size 1 1) (thickness 0.15)))
@@
     (property "Sheetname" "")
     (property "exclude_from_bom" "")
-    (attr through_hole exclude_from_bom)
+    (attr through_hole exclude_from_pos_files exclude_from_bom)
     (fp_text reference "J2" (at 0 -3.2) (layer "F.SilkS")
       (effects (font (size 1 1) (thickness 0.15)))
@@
     (pad "8" smd roundrect (at 2.8 -0.85 270) (size 0.5 1.1) (layers "B.Cu" "B.Paste" "B.Mask") (roundrect_rratio 0.25)
       (net 8 "/Display_CS") (pinfunction "Pin_8") (pintype "passive"))
-    (pad "MP" smd roundrect (at -4.1 0.55 270) (size 1.2 1.7) (layers "B.Cu" "B.Paste" "B.Mask") (roundrect_rratio 0.208333))
-    (pad "MP" smd roundrect (at 4.1 0.55 270) (size 1.2 1.7) (layers "B.Cu" "B.Paste" "B.Mask") (roundrect_rratio 0.208333))
+    (pad "MP" smd roundrect (at -4.1 0.55 270) (size 1.2 1.7) (layers "B.Cu" "B.Paste" "B.Mask") (roundrect_rratio 0.2083333333))
+    (pad "MP" smd roundrect (at 4.1 0.55 270) (size 1.2 1.7) (layers "B.Cu" "B.Paste" "B.Mask") (roundrect_rratio 0.2083333333))
     (model "${KICAD6_3DMODEL_DIR}/Connector_JST.3dshapes/JST_SUR_BM08B-SURS-TF_1x08-1MP_P0.80mm_Vertical.wrl"
       (offset (xyz 0 0 0))
@@
       ) (layer "B.SilkS") (width 0) (fill solid))
   )
+  (gr_circle (center 110.5 122.9) (end 110.723607 122.9) (layer "B.SilkS") (width 0.15) (fill solid))
   (gr_circle (center 116.3 154.9) (end 118.002939 154.9) (layer "F.SilkS") (width 0.15) (fill solid))
   (gr_circle (center 108.4 154.9) (end 110.102939 154.9) (layer "F.SilkS") (width 0.15) (fill solid))
@@
   (gr_line (start 126.4 90) (end 126.4 158.26) (layer "Edge.Cuts") (width 0.1))
   (gr_line (start 90 90) (end 126.4 90) (layer "Edge.Cuts") (width 0.1))
-  (gr_text "https://github.com/bablokb/pcb-pico-datalogger\nDisplay Adapter Rev. 0.90" (at 92.9 102.3 90) (layer "B.SilkS")
+  (gr_text "https://github.com/bablokb/pcb-pico-datalogger\nDisplay Adapter Rev. 1.00" (at 92.9 102.3 90) (layer "B.SilkS")
     (effects (font (size 1 1) (thickness 0.15)) (justify left mirror))
   )

Commit message: Display-Adaper Rev 1.10: add pin-headers to board (and production files)
Other:
- board text added: "https://github.com/bablokb/pcb-pico-datalogger Display Adapter Rev. 1.10"
- board text removed: "https://github.com/bablokb/pcb-pico-datalogger Display Adapter Rev. 1.00"
Changed lines of the file:
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@@
     (descr "Through hole straight pin header, 1x20, 2.54mm pitch, single row")
     (tags "Through hole pin header THT 1x20 2.54mm single row")
+    (property "LCSC" "C725952")
     (property "Sheetfile" "display_adapter.kicad_sch")
     (property "Sheetname" "")
-    (property "exclude_from_bom" "")
-    (attr through_hole exclude_from_pos_files exclude_from_bom)
+    (attr through_hole)
     (fp_text reference "J3" (at 0.4 51.55) (layer "F.SilkS")
       (effects (font (size 1 1) (thickness 0.15)))
@@
     (descr "Through hole straight pin header, 1x20, 2.54mm pitch, single row")
     (tags "Through hole pin header THT 1x20 2.54mm single row")
+    (property "LCSC" "C725952")
     (property "Sheetfile" "display_adapter.kicad_sch")
     (property "Sheetname" "")
-    (property "exclude_from_bom" "")
-    (attr through_hole exclude_from_pos_files exclude_from_bom)
+    (attr through_hole)
     (fp_text reference "J2" (at 0 -3.2) (layer "F.SilkS")
       (effects (font (size 1 1) (thickness 0.15)))
@@
     (property "Sheetname" "")
     (attr smd)
-    (fp_text reference "J1" (at 0 2.6 90) (layer "B.SilkS")
+    (fp_text reference "J1" (at 0 2.6 90) (layer "B.SilkS") hide
       (effects (font (size 1 1) (thickness 0.15)) (justify mirror))
     )
@@
   (gr_line (start 126.4 90) (end 126.4 158.26) (layer "Edge.Cuts") (width 0.1))
   (gr_line (start 90 90) (end 126.4 90) (layer "Edge.Cuts") (width 0.1))
-  (gr_text "https://github.com/bablokb/pcb-pico-datalogger\nDisplay Adapter Rev. 1.00" (at 92.9 102.3 90) (layer "B.SilkS")
+  (gr_text "CS" (at 104.109524 128.6) (layer "B.SilkS")
+    (effects (font (size 1 1) (thickness 0.15)) (justify right mirror))
+  )
+  (gr_text "3V3" (at 103.3 123) (layer "B.SilkS")
+    (effects (font (size 1 1) (thickness 0.15)) (justify right mirror))
+  )
+  (gr_text "https://github.com/bablokb/pcb-pico-datalogger\nDisplay Adapter Rev. 1.10" (at 92.9 102.3 90) (layer "B.SilkS")
     (effects (font (size 1 1) (thickness 0.15)) (justify left mirror))
   )
