File: display_adapter.kicad_sch (KiCad schematic)
At the start: 8 parts, among them J1 Conn_Display, J2 Inky_Left_1_20, J3 Inky_Right_21_40, J4 Ada_SPI_Display

Commit message: Display-Adaper Rev 1.10: add pin-headers to board (and production files)
Parts:
- J2, J3: LCSC (none) -> C725952; now in the parts list
Changed lines of the file:
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@@
   (title_block
     (title "Display-Adapter")
-    (date "2023-12-07")
-    (rev "1.00")
+    (date "2024-01-10")
+    (rev "1.10")
     (company "Bernhard Bablok")
     (comment 1 "https://github.com/bablokb/pcb-pico-datalogger")
@@
   )
   (symbol (lib_id "Connector_Generic:Conn_01x20") (at 114.808 61.468 0) (unit 1)
-    (in_bom no) (on_board yes)
+    (in_bom yes) (on_board yes)
     (property "Reference" "J2" (id 0) (at 112.268 25.908 0)
       (effects (font (size 1.27 1.27)) (justify left))
@@
     )
     (property "Datasheet" "~" (id 3) (at 114.808 61.468 0)
+      (effects (font (size 1.27 1.27)) hide)
+    )
+    (property "LCSC" "C725952" (id 4) (at 114.808 61.468 0)
       (effects (font (size 1.27 1.27)) hide)
     )
@@
   )
   (symbol (lib_id "Connector_Generic:Conn_01x20") (at 140.208 64.262 180) (unit 1)
-    (in_bom no) (on_board yes)
+    (in_bom yes) (on_board yes)
     (property "Reference" "J3" (id 0) (at 144.018 25.908 0)
       (effects (font (size 1.27 1.27)) (justify left))
@@
       (effects (font (size 1.27 1.27)) hide)
     )
+    (property "LCSC" "C725952" (id 4) (at 140.208 64.262 0)
+      (effects (font (size 1.27 1.27)) hide)
+    )
